File: kiCad/kiCad.kicad_pcb (KiCad board)
At the start: 2 copper layers, 111.1 x 88.9 mm, 32 parts, among them SW1 SW_Push, SW10 SW_Push, SW11 SW_Push, SW12 SW_Push, SW2 SW_Push, SW3 SW_Push, SW4 SW_Push, SW5 SW_Push, SW6 SW_Push, SW7 SW_Push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

Commit message: Board routed but missing OLED screen, corner chamfers, mounting holes, logo, and switch footprint fix.
Parts:
- moved R4 24.2 mm to (103.5, 76.7), turned to 0 degrees
Routing:
- net /COL0: track 0.00 -> 142.5 mm
- net /COL1: track 0.00 -> 140.7 mm
- net /ROW3: track 0.00 -> 136.7 mm
- net /COL2: track 0.00 -> 96.6 mm
- net /ROW0: track 0.00 -> 95.8 mm
- net /ROW2: track 0.00 -> 82.8 mm
- net VCC: track 0.00 -> 75.7 mm
- net /ROW1: track 0.00 -> 73.2 mm
- net /EN_CLK: track 0.00 -> 53.5 mm
- net Net-(R5-Pad2): track 0.00 -> 33.1 mm
- net Net-(R4-Pad2): track 0.00 -> 15.1 mm
- net Net-(D4-Pad2): track 0.00 -> 7.25 mm
- net Net-(D3-Pad2): track 0.00 -> 7.25 mm
- net Net-(D2-Pad2): track 0.00 -> 7.25 mm
- net Net-(D12-Pad2): track 0.00 -> 7.25 mm
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- added copper zone on B.Cu, net GND
- added copper zone on F.Cu, net GND

Commit message: Updated the switch footprints, chamfered corners, added mounting holes. Still need to add logo, but then it'll be ready for manufacturing.
Parts:
- added G1: thinOLED, keyboardLib:thinOLED, F.Cu at (113.6, 37.9)
- added REF**: MountingHole_2.7mm, MountingHole:MountingHole_2.7mm, F.Cu at (133.3, 28.6)
- added REF**: MountingHole_2.7mm, MountingHole:MountingHole_2.7mm, F.Cu at (28.6, 111.1)
- added REF**: MountingHole_2.7mm, MountingHole:MountingHole_2.7mm, F.Cu at (28.6, 28.6)
- added REF**: MountingHole_2.7mm, MountingHole:MountingHole_2.7mm, F.Cu at (133.3, 111.1)
Connections:
- U1 pad 5: Net-(U1-Pad5) -> /SDA
- U1 pad 6: Net-(U1-Pad6) -> /SCL
Routing:
- net VCC: track 75.7 -> 129.3 mm
- net /SDA: track 0.00 -> 28.8 mm
- net /SCL: track 0.00 -> 25.2 mm
- net /COL0: track 142.5 -> 143.6 mm
Other:
- outline, holes or cut-outs redrawn

Commit message: Added logo to solder mask layer (will show the underlying copper fill there). Sending out for manufacturing.
Parts:
- added G***: LOGO, Logo:logo, F.Cu at (60.3, 29.2)
